Commit message: yippie

File: description/robot.urdf.xacro (robot description, xacro)
@@ -4,3 +4,4 @@
     <xacro:include filename="inertial_macros.xacro" />
     <xacro:include filename="lidar.xacro" />
+    <xacro:include filename="gazebo.xacro" />
 </robot>

File: description/robot_core.xacro (robot description, xacro)
@@ -264,84 +264,3 @@
     <dynamics damping="0.1" friction="0.1"/>
   </joint>
-  <!-- Gazebo Parameters -->
-  <gazebo reference="body_link">
-    <mu1>0.0001</mu1>
-    <mu2>0.0001</mu2>
-  </gazebo>
-  <gazebo reference="front_right_wheel_link">
-    <mu1>100.0</mu1>
-    <mu2>100.0</mu2>
-  </gazebo>
-  <gazebo reference="front_left_wheel_link">
-    <mu1>100.0</mu1>
-    <mu2>100.0</mu2>
-  </gazebo>
-  <gazebo reference="rear_right_wheel_link">
-    <mu1>100.0</mu1>
-    <mu2>100.0</mu2>
-  </gazebo>
-  <gazebo reference="rear_left_wheel_link">
-    <mu1>100.0</mu1>
-    <mu2>100.0</mu2>
-  </gazebo>
-  <!-- Gazebo Control -->
-  <ros2_control name="control" type="system">
-    <hardware>
-      <plugin>gz_ros2_control/GazeboSimSystem</plugin>
-    </hardware>
-    <joint name="front_left_steering_joint">
-      <command_interface name="position">
-        <param name="min">${-max_steering_angle}</param>
-        <param name="max">${max_steering_angle}</param>
-      </command_interface>
-      <state_interface name="position"/>
-      <state_interface name="velocity"/>
-      <state_interface name="effort"/>
-    </joint>
-    <joint name="front_right_steering_joint">
-      <command_interface name="position">
-        <param name="min">${-max_steering_angle}</param>
-        <param name="max">${max_steering_angle}</param>
-      </command_interface>
-      <state_interface name="position"/>
-      <state_interface name="velocity"/>
-      <state_interface name="effort"/>
-    </joint>
-    <joint name="rear_left_wheel_joint">
-      <command_interface name="velocity">
-        <param name="min">${-max_wheel_angular_velocity}</param>
-        <param name="max">${max_wheel_angular_velocity}</param>
-      </command_interface>
-      <state_interface name="position"/>
-      <state_interface name="velocity"/>
-      <state_interface name="effort"/>
-    </joint>
-    <joint name="rear_right_wheel_joint">
-      <command_interface name="velocity">
-        <param name="min">${-max_wheel_angular_velocity}</param>
-        <param name="max">${max_wheel_angular_velocity}</param>
-      </command_interface>
-      <state_interface name="position"/>
-      <state_interface name="velocity"/>
-      <state_interface name="effort"/>
-    </joint>
-  </ros2_control>
-  <!-- Gazebo Plugins -->
-  <gazebo>
-    <plugin filename="gz-sim-joint-state-publisher-system" name="gz::sim::systems::JointStatePublisher">
-      <topic>joint_states</topic>
-      <joint_name>front_left_steering_joint</joint_name>
-      <joint_name>front_right_steering_joint</joint_name>
-      <joint_name>front_left_wheel_joint</joint_name>
-      <joint_name>front_right_wheel_joint</joint_name>
-      <joint_name>rear_left_wheel_joint</joint_name>
-      <joint_name>rear_right_wheel_joint</joint_name>
-    </plugin>
-    <plugin filename="gz_ros2_control-system" name="gz_ros2_control::GazeboSimROS2ControlPlugin">
-      <parameters>$(find my_bot)/config/gz_ros2_control.yaml</parameters>
-    </plugin>
-    <plugin filename="gz-sim-sensors-system" name="gz::sim::systems::Sensors">
-      <render_engine>ogre2</render_engine>
-    </plugin>
-  </gazebo>
 </robot>
